Commit message: rover-teleop-bridge successfull setup

File: urdf/rover.urdf (robot description, URDF)
Before this commit: robot mars_rover, 18 links, 17 joints
Links:
- removed link camera_link
- removed link camera_link_1
- removed link camera_link_2
- removed link camera_optical_link
- removed link camera_optical_link_1
- removed link camera_optical_link_2
- removed link imu_link
- link chassis: geometry collision mesh filename=file://$(find rover_control)/meshes/base_link.STL; visual mesh filename=file://$(find rover_control)/meshes/base_link.STL
- link steering1: geometry collision mesh filename=file://$(find rover_control)/meshes/steering1.STL; visual mesh filename=file://$(find rover_control)/meshes/steering1.STL
- link steering2: geometry collision mesh filename=file://$(find rover_control)/meshes/steering2.STL; visual mesh filename=file://$(find rover_control)/meshes/steering2.STL
- link steering3: geometry collision mesh filename=file://$(find rover_control)/meshes/steering3.STL; visual mesh filename=file://$(find rover_control)/meshes/steering3.STL
- link steering4: geometry collision mesh filename=file://$(find rover_control)/meshes/steering4.STL; visual mesh filename=file://$(find rover_control)/meshes/steering4.STL
- link wheel1: geometry collision cylinder length=0.144 radius=0.11; visual mesh filename=file://$(find rover_control)/meshes/wheel1.STL
- link wheel2: geometry collision cylinder length=0.144 radius=0.11; visual mesh filename=file://$(find rover_control)/meshes/wheel2.STL
- link wheel3: geometry collision cylinder length=0.144 radius=0.11; visual mesh filename=file://$(find rover_control)/meshes/wheel3.STL
- link wheel4: geometry collision cylinder length=0.144 radius=0.11; visual mesh filename=file://$(find rover_control)/meshes/wheel4.STL
Joints:
- removed joint camera_joint
- removed joint camera_joint_1
- removed joint camera_joint_2
- removed joint camera_optical_joint
- removed joint camera_optical_joint_1
- removed joint camera_optical_joint_2
- removed joint imu_joint
